Commit message: new

File: src/medipick_simple3_description/urdf/simple3_moveit.urdf (robot description, URDF)
Before this commit: robot simple4_urdf, 16 links, 15 joints
Links:
- removed link base_roll_link
- added link base_body_link, mass 26.422; collision mesh filename=package://medipick_simple3_description/vendor/simple5_curre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; visual mesh filename=package://medipick_simple3_description/vendor/simple5_curre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
- added link base_imu_link, mass 0.001
- added link cam_link, mass 0.012566; visual box size=0.004 0.040 0.024; visual box size=0.016 0.018 0.042
- added link cam_sensor_link, mass 0.001
- added link sucker_contact_link, mass 0.0001
- link base_link: mass 26.422 -> 0.001; geometry 
- link h1_link: mass 0.064115 -> 0.087226; geometry collision mesh filename=package://medipick_simple3_description/vendor/simple5_curre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; visual mesh filename=package://medipick_simple3_description/vendor/simple5_curre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
- link h2_link: mass 0.081692 -> 0.017576; geometry collision mesh filename=package://medipick_simple3_description/vendor/simple5_curre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; visual mesh filename=package://medipick_simple3_description/vendor/simple5_curre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
- link r1_link: geometry collision mesh filename=package://medipick_simple3_description/vendor/simple5_curre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; visual mesh filename=package://medipick_simple3_description/vendor/simple5_curre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
- link r2_link: geometry collision mesh filename=package://medipick_simple3_description/vendor/simple5_curre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; visual mesh filename=package://medipick_simple3_description/vendor/simple5_curre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
- link r3_link: geometry collision mesh filename=package://medipick_simple3_description/vendor/simple5_curre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; visual mesh filename=package://medipick_simple3_description/vendor/simple5_curre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
- link r4_link: geometry collision mesh filename=package://medipick_simple3_description/vendor/simple5_curre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; visual mesh filename=package://medipick_simple3_description/vendor/simple5_curre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
- link r5_link: geometry collision mesh filename=package://medipick_simple3_description/vendor/simple5_curre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; visual mesh filename=package://medipick_simple3_description/vendor/simple5_curre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
- link r6_link: geometry collision mesh filename=package://medipick_simple3_description/vendor/simple5_curre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; visual mesh filename=package://medipick_simple3_description/vendor/simple5_curre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
- link raise_link: mass 1.4841 -> 1.2939; geometry collision mesh filename=package://medipick_simple3_description/vendor/simple5_curre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; visual mesh filename=package://medipick_simple3_description/vendor/simple5_curre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
- link sucker_link: geometry collision mesh filename=package://medipick_simple3_description/vendor/simple5_curre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; visual mesh filename=package://medipick_simple3_description/vendor/simple5_curre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
Joints:
- removed joint base_heading_mount
- removed joint base_roll_mount
- added joint base_body_mount: type fixed, parent base_link, child base_body_link, origin xyz=0 0 0 rpy=3.141592653589793 0 -1.5707963267948966
- added joint base_imu_mount: type fixed, parent base_link, child base_imu_link, origin xyz=0 0 0 rpy=0 0 0
- added joint base_mount: type fixed, parent base_theta_link, child base_link, origin xyz=0 0 0 rpy=0 0 0
- added joint cam_joint: type fixed, parent h2_link, child cam_link, origin xyz=0.0181 -0.067717 -0.043841 rpy=3.141592653589793 -0.5236 -1.5708
- added joint cam_sensor_joint: type fixed, parent cam_link, child cam_sensor_link, origin xyz=0.052 0 0 rpy=0 0 0
- added joint sucker_contact_joint: type fixed, parent sucker_link, child sucker_contact_link, origin xyz=0.0428 0 0 rpy=0 0 0
- joint base_theta: limit lower=-3.141592653589793 upper=3.141592653589793 effort=150.0 velocity=1.57 -> effort=150.0 velocity=3.14; type revolute -> continuous
- joint base_x: limit lower=-3.0 upper=3.0 effort=400.0 velocity=1.0 -> lower=-100.0 upper=100.0 effort=400.0 velocity=2.0
- joint base_y: limit lower=-3.0 upper=3.0 effort=400.0 velocity=1.0 -> lower=-100.0 upper=100.0 effort=400.0 velocity=2.0
- joint h1_joint: axis 0 0 1 -> 0 0 -1; origin xyz=0 -0.125 -0.0489 rpy=0 0 0 -> xyz=0 -0.125 0.0261 rpy=0 0 0
- joint r1_joint: origin xyz=0.061 -0.125 0.064068 rpy=0 0 0 -> xyz=0.061 -0.125 0.13907 rpy=0 0 0
- joint raise_joint: limit lower=0.0 upper=1.5 effort=100.0 velocity=0.2 -> lower=0.0 upper=1.5 effort=2500.0 velocity=0.4; origin xyz=0 0 -0.939 rpy=0 0 0 -> xyz=0 0 -0.97 rpy=0 0 0; parent base_link -> base_body_link
